File: backplane.kicad_pcb (KiCad board)
At the start: 2 copper layers, 93.9 x 83.8 mm, 67 parts, among them J1 I2C, J2 I2C, J3 SER, J4 PWR, J5 PWR, J6 FAN, Q1 Q_NMOS_GSD, Q2 Q_NMOS_GSD, Q3 Q_NMOS_GSD, Q4 Q_NMOS_GSD, Q5 Q_PMOS_GSD, SW1 SW_Push, U1 Raspberry_Pi_2_3, U2 IC880A-SPI, U3 SHT21, U4 MP1584_MODULE, U5 MCP3425A0T-E/CH

Commit message: Remove labels
Parts:
- removed G***: LOGO, oshw-logos:OSHW_MASK_7MM
Other:
- board text removed: "OSHW"
- board text removed: "coredump.ch / adnexo.ch 2017"
- board text removed: "https://github.com/dbrgn/ic880a-backplane"
- board text removed: "iC880A Backplane v1.2"
